File: 60_case_keyboard/60_case_keyboard.kicad_pcb (KiCad board)
At the start: 2 copper layers, 285 x 95.1 mm, 119 parts, among them IC1 REG71050DDCR, J1 BATT_CONN, J2 PROG_CONN, Q1 AO3407, SW1 BATT_SWITCH, SW10 SW_Push, SW11 SW_Push, SW12 SW_Push, SW13 SW_Push, SW14 SW_Push, SW15 SW_Push, SW16 SW_Push, SW17 SW_Push, SW18 SW_Push, SW19 SW_Push, SW2 SW_Push, SW20 SW_Push, SW21 SW_Push, SW22 SW_Push, SW23 SW_Push, SW24 SW_Push, SW25 SW_Push, SW26 SW_Push, SW27 SW_Push, SW28 SW_Push, SW29 SW_Push, SW3 SW_Push, SW30 SW_Push, SW31 SW_Push, SW32 SW_Push, SW33 SW_Push, SW34 SW_Push, SW35 SW_Push, SW36 SW_Push, SW37 SW_Push, SW38 Rotary_Encoder_Switch, SW4 SW_Push, SW5 SW_Push, SW6 SW_Push, SW7 SW_Push, SW8 SW_Push, SW9 SW_Push, U1 E73-2G4M08S1C, U2 MCP73831, U3 AP2112K-3.3, U4 LS027B7DH01, Y1 32.768kHz

Commit message: Info on flashing
Parts:
- added REF**: OSHW-Logo2_14.6x12mm_SilkScreen, Symbol:OSHW-Logo2_14.6x12mm_SilkScreen, B.Cu at (63.2, 148.5)
Routing:
- net GND: track 690.3 -> 67.8 mm, vias 10 -> 1
- net R_ENCODER_B: track 133.5 -> 126.7 mm
- net COL09: track 216.4 -> 214.1 mm, vias 0 -> 1
- net R_ENCODER_A: track 136.2 -> 134.4 mm
- net R_ENCODER_SWITCH: track 125.9 -> 124.3 mm
- net Net-(D19-Pad2): track 54.2 -> 55.3 mm, vias 0 -> 2
- net COL08: track 218.8 -> 218.2 mm
- net COL07: track 169.2 -> 168.7 mm
- net Net-(D20-Pad2): track 38.3 -> 37.8 mm, vias 0 -> 1
- net Net-(D18-Pad2): vias 0 -> 2
- added copper zone on B.Cu, net GND
- added copper zone on F.Cu, net GND
Other:
- board text added: "JLCJLCJLCJLC"
